Commit message: change names of links and joints around gripper

File: nekonote_description/urdf/end_effector_A/end_effector_A.xacro (robot description, xacro)
@@ -5,5 +5,5 @@
   <xacro:macro name="end_effector_A" params="prefix">
     <!-- links -->
-    <link name="${prefix}hand1">
+    <link name="${prefix}gripper_base">
       <visual>
         <origin xyz="0 0 0" rpy="0 0 0"/>
@@ -25,5 +25,5 @@
       </inertial>
     </link>
-    <link name="${prefix}hand2">
+    <link name="${prefix}gripper_finger">
       <visual>
         <origin xyz="0 0 0" rpy="${m_pi_2} 0 0"/>
@@ -47,21 +47,21 @@
     <link name="${prefix}tool0"/>
     <!-- joints -->
-    <joint name="${prefix}hand_base-hand1" type="fixed">
+    <joint name="${prefix}hand_base-gripper_base" type="fixed">
       <origin xyz="0 0 0" rpy="0 0 0"/>
       <parent link="${prefix}hand_base"/>
-      <child link="${prefix}hand1"/>
+      <child link="${prefix}gripper_base"/>
       <axis xyz="0 0 1"/>
     </joint>
-    <joint name="${prefix}hand_joint" type="revolute">
+    <joint name="${prefix}gripper_joint" type="revolute">
       <origin xyz="0.004 0 0.0155" rpy="0 0 0"/>
-      <parent link="${prefix}hand1"/>
-      <child link="${prefix}hand2"/>
+      <parent link="${prefix}gripper_base"/>
+      <child link="${prefix}gripper_finger"/>
       <axis xyz="0 1 0"/>
       <limit lower="0.01658" upper="1.1576" effort="0" velocity="0"/>
     </joint>
-    <joint name="${prefix}hand2-tool0" type="fixed">
+    <joint name="${prefix}gripper_finger-tool0" type="fixed">
       <!-- TODO fix tool0 position-->
       <origin xyz="0 0 0.01" rpy="0 0 0" />
-      <parent link="${prefix}hand2"/>
+      <parent link="${prefix}gripper_finger"/>
       <child link="${prefix}tool0"/>
     </joint>

File: nekonote_description/urdf/nekonote.urdf (robot description, URDF)
Before this commit: robot nekonote, 11 links, 10 joints
Links:
- removed link hand1
- removed link hand2
- added link gripper_base, mass 0.094464; collision mesh filename=package://nekonote_description/meshes/collision/end_effecto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; visual mesh filename=package://nekonote_description/meshes/visual/end_effector_A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
- added link gripper_finger, mass 0.023997; collision mesh filename=package://nekonote_description/meshes/collision/end_effecto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; visual mesh filename=package://nekonote_description/meshes/visual/end_effector_A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
Joints:
- removed joint hand2-tool0
- removed joint hand_base-hand1
- removed joint hand_joint
- added joint gripper_finger-tool0: type fixed, parent gripper_finger, child tool0, origin xyz=0 0 0.01 rpy=0 0 0
- added joint gripper_joint: type revolute, parent gripper_base, child gripper_finger, origin xyz=0.004 0 0.0155 rpy=0 0 0, axis 0 1 0, limit lower=0.01658 upper=1.1576 effort=0 velocity=0
- added joint hand_base-gripper_base: type fixed, parent hand_base, child gripper_base, origin xyz=0 0 0 rpy=0 0 0, axis 0 0 1
