Commit message: reduce polygon counts of models

File: nekonote_description/urdf/base/base.urdf.xacro (robot description, xacro)
@@ -5,5 +5,5 @@
   <xacro:macro name="nekonote_base" params="prefix">
     <!-- links -->
-    <link name="${prefix}base" />
+    <link name="${prefix}base"/>
     <link name="${prefix}base_link">
       <visual>
@@ -129,7 +129,7 @@
     <!-- joints -->
     <joint name="${prefix}base_link-base" type="fixed">
-      <parent link="${prefix}base_link" />
-      <child link="${prefix}base" />
-      <origin xyz="0 0 0" rpy="0 0 0" />
+      <origin xyz="0 0 0" rpy="0 0 0"/>
+      <parent link="${prefix}base_link"/>
+      <child link="${prefix}base"/>
     </joint>
     <joint name="${prefix}joint0" type="revolute">

File: nekonote_description/urdf/common_materials.xacro (robot description, xacro)
@@ -3,5 +3,5 @@
   <xacro:macro name="material_grey">
     <material name="">
-      <color rgba=".1 .1 .1 1"/>
+      <color rgba="0.3 0.3 0.3 1"/>
     </material>
   </xacro:macro>

Commit message: add the acurate tool0 frame and effort limits of joints to URDF

File: nekonote_description/urdf/base/base.urdf.xacro (robot description, xacro)
@@ -138,5 +138,5 @@
       <child link="${prefix}link1"/>
       <axis xyz="0 0 1"/>
-      <limit lower="-1.7453" upper="1.7453" effort="0" velocity="0"/>
+      <limit lower="-1.7453" upper="1.7453" effort="5" velocity="0"/>
     </joint>
     <joint name="${prefix}joint1" type="revolute">
@@ -145,5 +145,5 @@
       <child link="${prefix}link2"/>
       <axis xyz="0 1 0"/>
-      <limit lower="-1.57" upper="1.57" effort="0" velocity="0"/>
+      <limit lower="-1.57" upper="1.57" effort="10" velocity="0"/>
     </joint>
     <joint name="${prefix}joint2" type="revolute">
@@ -152,5 +152,5 @@
       <child link="${prefix}link3"/>
       <axis xyz="0 1 0"/>
-      <limit lower="-1.8353" upper="2.5837" effort="0" velocity="0"/>
+      <limit lower="-1.8353" upper="2.5837" effort="5" velocity="0"/>
     </joint>
     <joint name="${prefix}joint3" type="revolute">
@@ -159,5 +159,5 @@
       <child link="${prefix}link4"/>
       <axis xyz="0 0 1"/>
-      <limit lower="-1.7453" upper="1.7453" effort="0" velocity="0"/>
+      <limit lower="-1.7453" upper="1.7453" effort="5" velocity="0"/>
     </joint>
     <joint name="${prefix}joint4" type="revolute">
@@ -166,5 +166,5 @@
       <child link="${prefix}link5"/>
       <axis xyz="0 -1 0"/>
-      <limit lower="-1.57" upper="1.57" effort="0" velocity="0"/>
+      <limit lower="-1.57" upper="1.57" effort="5" velocity="0"/>
     </joint>
     <joint name="${prefix}joint5" type="revolute">
@@ -173,5 +173,5 @@
       <child link="${prefix}hand_base"/>
       <axis xyz="0 0 -1"/>
-      <limit lower="-1.7453" upper="1.7453" effort="0" velocity="0"/>
+      <limit lower="-1.7453" upper="1.7453" effort="5" velocity="0"/>
     </joint>
   </xacro:macro>

File: nekonote_description/urdf/end_effector_A/end_effector_A.xacro (robot description, xacro)
@@ -60,8 +60,7 @@
       <limit lower="0.01658" upper="1.1576" effort="0" velocity="0"/>
     </joint>
-    <joint name="${prefix}gripper_finger-tool0" type="fixed">
-      <!-- TODO fix tool0 position-->
-      <origin xyz="0 0 0.01" rpy="0 0 0" />
-      <parent link="${prefix}gripper_finger"/>
+    <joint name="${prefix}gripper_base-tool0" type="fixed">
+      <origin xyz="0 0 0.08" rpy="0 0 0" />
+      <parent link="${prefix}gripper_base"/>
       <child link="${prefix}tool0"/>
     </joint>

File: nekonote_description/urdf/nekonote.urdf (robot description, URDF)
Before this commit: robot nekonote, 11 links, 10 joints
Joints:
- removed joint gripper_finger-tool0
- added joint gripper_base-tool0: type fixed, parent gripper_base, child tool0, origin xyz=0 0 0.08 rpy=0 0 0
- joint joint0: limit lower=-1.7453 upper=1.7453 effort=0 velocity=0 -> lower=-1.7453 upper=1.7453 effort=5 velocity=0
- joint joint1: limit lower=-1.57 upper=1.57 effort=0 velocity=0 -> lower=-1.57 upper=1.57 effort=10 velocity=0
- joint joint2: limit lower=-1.8353 upper=2.5837 effort=0 velocity=0 -> lower=-1.8353 upper=2.5837 effort=5 velocity=0
- joint joint3: limit lower=-1.7453 upper=1.7453 effort=0 velocity=0 -> lower=-1.7453 upper=1.7453 effort=5 velocity=0
- joint joint4: limit lower=-1.57 upper=1.57 effort=0 velocity=0 -> lower=-1.57 upper=1.57 effort=5 velocity=0
- joint joint5: limit lower=-1.7453 upper=1.7453 effort=0 velocity=0 -> lower=-1.7453 upper=1.7453 effort=5 velocity=0

Commit message: fix the rotation direction of joint3

File: nekonote_description/urdf/base/base.urdf.xacro (robot description, xacro)
@@ -158,5 +158,5 @@
       <parent link="${prefix}link3"/>
       <child link="${prefix}link4"/>
-      <axis xyz="0 0 1"/>
+      <axis xyz="0 0 -1"/>
       <limit lower="-1.7453" upper="1.7453" effort="5" velocity="0"/>
     </joint>

File: nekonote_description/urdf/nekonote.urdf (robot description, URDF)
Before this commit: robot nekonote, 11 links, 10 joints
Joints:
- joint joint3: axis 0 0 1 -> 0 0 -1
